File: power_5.0.kicad_sch (KiCad schematic)
At the start: 3 parts

Commit message: schematic completed
Parts:
- gave numbers to parts that had none: 3
Changed lines of the file:
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@@
 		(dnp no)
 		(fields_autoplaced yes)
-		(property "Reference" "C?"
+		(property "Reference" "C5"
 			(at 120.65 81.28 90)
 			(show_name no)
@@
 			(project "cansat-2026"
 				(path "/e7460e48-0dfd-427c-9e44-f917ebe6a296/87bdd923-3d33-4a25-9c4e-e3464401770b"
-					(reference "C?")
+					(reference "C7")
 					(unit 1)
 				)
 				(path "/e7460e48-0dfd-427c-9e44-f917ebe6a296/cac25c5d-e21e-4cd3-87ea-c3eb3e0053b1"
-					(reference "C?")
+					(reference "C5")
 					(unit 1)
 				)
@@
 		(dnp no)
 		(fields_autoplaced yes)
-		(property "Reference" "U?"
+		(property "Reference" "U3"
 			(at 157.48 82.4798 0)
 			(show_name no)
@@
 			(project "cansat-2026"
 				(path "/e7460e48-0dfd-427c-9e44-f917ebe6a296/87bdd923-3d33-4a25-9c4e-e3464401770b"
-					(reference "U?")
+					(reference "U4")
 					(unit 1)
 				)
 				(path "/e7460e48-0dfd-427c-9e44-f917ebe6a296/cac25c5d-e21e-4cd3-87ea-c3eb3e0053b1"
-					(reference "U?")
+					(reference "U3")
 					(unit 1)
 				)
@@
 		(dnp no)
 		(fields_autoplaced yes)
-		(property "Reference" "C?"
+		(property "Reference" "C6"
 			(at 160.02 93.9799 0)
 			(show_name no)
@@
 			(project "cansat-2026"
 				(path "/e7460e48-0dfd-427c-9e44-f917ebe6a296/87bdd923-3d33-4a25-9c4e-e3464401770b"
-					(reference "C?")
+					(reference "C8")
 					(unit 1)
 				)
 				(path "/e7460e48-0dfd-427c-9e44-f917ebe6a296/cac25c5d-e21e-4cd3-87ea-c3eb3e0053b1"
-					(reference "C?")
-					(unit 1)
-				)
+					(reference "C6")
+					(unit 1)
+				)
