File: cansat-2026.kicad_pcb (KiCad board)
At the start: 4 copper layers, 35 x 80 mm, 46 parts, among them J1 AE-S8474-TX, J2 AE-S8474-TX, J3 UART, J4 tx_coil, M1 Motor_DC, M2 Motor_DC, M3 Motor_Servo, M4 Motor_Servo, Q1 Q_Photo_NPN_EC, Q2 Q_NPN_BEC, Q3 Q_PMOS_GDS, U1 TPM8837C, U2 TPM8837C, U3 MYRBPxx0080B21RD, U4 MYRBPxx0080B21RD

Commit message: wip (wiring)
Parts:
- moved C1 18.8 mm to (6.91, 60.1)
- moved R1 3.57 mm to (16.3, 26.0), turned to -90 degrees
Connections:
- A1 pad 35: /3V3 -> unconnected-(A1-ADC_VREF-Pad35)
- R5 pad 1: /Sol -> /V_{Sol}
Routing:
- net /V_{M}: track 0.00 -> 100.3 mm, vias 0 -> 24
- net /3V3: track 0.00 -> 69.1 mm
- net /V_{Lipo}: track 0.00 -> 57.3 mm, vias 0 -> 9
- net /V_{Sol}: track 0.00 -> 46.1 mm, vias 0 -> 1
- net /M1_EN: track 0.00 -> 43.6 mm, vias 0 -> 3
- net GND: track 0.00 -> 25.0 mm, vias 0 -> 9
- net /IMU_RESET: track 0.00 -> 14.4 mm
- net /IMU_INT: track 0.00 -> 14.0 mm
- net /Servo_IN: track 0.00 -> 11.2 mm
- net /PServo_IN: track 0.00 -> 10.8 mm
- net /M2_OUT1: track 0.00 -> 10.7 mm
- net /M1_OUT1: track 0.00 -> 9.89 mm
- net /M1_OUT2: track 0.00 -> 9.63 mm
- net /I2C1_SCL: track 0.00 -> 9.47 mm
- net /I2C1_SDA: track 0.00 -> 9.47 mm
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- added copper zone on F.Cu, net /V_{Lipo}
- added copper zone on F.Cu, net /V_{M}
- added copper zone on In2.Cu, net /V_{M}
- added copper zone on In1.Cu, net GND
- added copper zone on B.Cu, net Net-(U3-L2)
- added copper zone on F.Cu, net Net-(U3-L2)
- added copper zone on B.Cu, net Net-(U4-L2)
- added copper zone on F.Cu, net Net-(U4-L2)

Commit message: finished wiring
Routing:
- net /V_{M}: track 100.3 -> 156.3 mm, vias 24 -> 18
- net /3V3: track 69.1 -> 72.1 mm
- net GND: track 25.0 -> 28.0 mm, vias 9 -> 11
- net /M2_OUT1: track 10.7 -> 9.72 mm
