File: cansat-2026.kicad_sch (KiCad schematic)
At the start: 34 parts

Commit message: schematic completed
Parts:
- removed Q?: NPN, symbol Simulation_SPICE:NPN
- removed Q?: PMOS, symbol Simulation_SPICE:PMOS
- added J3: UART, Connector_PinHeader_2.54mm:PinHeader_1x03_P2.54mm_Vertical, symbol Connector:Conn_01x03_Pin
- added Q2: Q_NPN_BEC, Package_TO_SOT_SMD:SOT-23-3, symbol Transistor_BJT:Q_NPN_BEC
- added Q3: Q_PMOS_GDS, Package_TO_SOT_SMD:TO-252-2, symbol Transistor_FET:Q_PMOS_GDS
- BT1: renamed from BT?; footprint (none) -> Connector_JST:JST_PH_B2B-PH-K_1x02_P2.00mm_Vertical
- C1: renamed from C?; value C -> 220u; footprint (none) -> Capacitor_THT:C_Radial_D8.0mm_H7.0mm_P3.50mm
- C2, C3: renamed from C?; value C -> 10u
- R1: renamed from R?; value R -> 10k; footprint Resistor_SMD:R_0603_1608Metric_Pad0.98x0.95mm_HandSolder -> Resistor_SMD:R_0603_1608Metric
- R10, R11, R12, R13, R14, R15, R3, R4: renamed from R?; footprint Resistor_SMD:R_0603_1608Metric_Pad0.98x0.95mm_HandSolder -> Resistor_SMD:R_0603_1608Metric
- R2: renamed from R?; value R -> 33k
- R7: renamed from R?; value R -> 470
- R8, R9: renamed from R?; value R -> 10k
- gave numbers to parts that had none: 15
Connections:
- net GND: now also J3.2 (Pin_2), Q2.2 (E)
- net UART0_RX: now also J3.3 (Pin_3)
- net UART0_TX: now also J3.1 (Pin_1)
- net V_{Sol}: now also Q3.3 (S)
- net WPT_V_{IN}: now also Q3.2 (D)
- net at R7.2: now also Q2.1 (B)
- net at R9.2: now also Q2.3 (C)
- net at R8.2, R9.1: now also Q3.1 (G)
Other:
- note added: "47"
- company: (none) -> NIT Gifu College - SERA
- title: (none) -> CanSat 2026 Main Board
- moved on the sheet: C1, C2, C3

Commit message: component placed
Parts:
- removed A1: RaspberryPi_Pico_W, Module:RaspberryPi_Pico_W_SMD_HandSolder, symbol MCU_Module:RaspberryPi_Pico_W_Debug
- added A1: RaspberryPi_Pico_W, Module:RaspberryPi_Pico_Common_THT, symbol MCU_Module:RaspberryPi_Pico_W
- added H1, H2, H3, H4: MountingHole, MountingHole:MountingHole_3.2mm_M3, symbol Mechanical:MountingHole
- added J4: tx_coil, Connector_PinSocket_2.54mm:PinSocket_1x02_P2.54mm_Vertical, symbol Connector:Conn_01x02_Pin
Connections:
- net WPT_GND is gone; now on net GND: J1.2 (Pin_2), J2.3 (Pin_3)
- net 3V3: now also A1.35 (ADC_VREF), A1.36 (3V3)
- net GEN_LVL: now also A1.31 (GPIO26_ADC0)
- net GND: now also A1.13 (GND), A1.18 (GND), A1.23 (GND), A1.28 (GND), A1.3 (GND), A1.33 (AGND), A1.38 (GND), A1.8 (GND)
- net I2C1_SCL: now also A1.10 (GPIO7)
- net I2C1_SDA: now also A1.9 (GPIO6)
- net IMU_INT: now also A1.7 (GPIO5)
- net IMU_RESET: now also A1.6 (GPIO4)
- net LIGHT_LVL: now also A1.32 (GPIO27_ADC1)
- net M1_EN: now also A1.19 (GPIO14)
- net UART0_RX: now also A1.2 (GPIO1)
- net UART0_TX: now also A1.1 (GPIO0)
- net VSYS: now also A1.39 (VSYS)
- net WPT_EN: now also A1.20 (GPIO15)
- net WPT_L+: now also J4.1 (Pin_1)
- net WPT_L-: now also J4.2 (Pin_2)
- net at R10.1: now also A1.11 (GPIO8)
- net at R11.1: now also A1.12 (GPIO9)
- net at R12.1: now also A1.14 (GPIO10)
- net at R13.1: now also A1.15 (GPIO11)
- net at R14.1: now also A1.16 (GPIO12)
- net at R15.1: now also A1.17 (GPIO13)

Commit message: wip (wiring)
Connections:
- net Sol is gone; now on net V_{Sol}: R5.1
- net 3V3: no longer A1.35 (ADC_VREF)
- no-connect marks 14 -> 15
Changed lines of the file:
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@@
+	)
+	(no_connect
+		(at 247.65 76.2)
 	)
 	(no_connect
@@
 		)
 	)
-	(label "3V3"
-		(at 247.65 76.2 0)
-		(effects
-			(font
-				(size 1.27 1.27)
-			)
-			(justify left bottom)
-		)
-	)
 	(label "M2_OUT2"
 		(at 214.63 152.4 270)
@@
 		)
 	)
-	(label "Sol"
-		(at 105.41 81.28 180)
-		(effects
-			(font
-				(size 1.27 1.27)
-			)
-			(justify right bottom)
-		)
-	)
 	(label "WPT_EN"
 		(at 132.08 96.52 180)
@@
 		)
 	)
+	(label "V_{Sol}"
+		(at 105.41 81.28 0)
+		(effects
+			(font
+				(size 1.27 1.27)
+			)
+			(justify left bottom)
+		)
+	)

Commit message: param modification
Parts:
- R2: value 33k -> 10k
- R3, R4: now not fitted
- R8: value 10k -> 100k
Changed lines of the file:
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@@
 		(on_board yes)
 		(in_pos_files yes)
-		(dnp no)
+		(dnp yes)
 		(fields_autoplaced yes)
 		(property "Reference" "R3"
@@
 			)
 		)
-		(property "Value" "10k"
+		(property "Value" "100k"
 			(at 152.4 73.6599 0)
 			(show_name no)
@@
 			)
 		)
-		(property "Value" "33k"
+		(property "Value" "10k"
 			(at 80.01 101.5999 0)
 			(show_name no)
@@
 		(on_board yes)
 		(in_pos_files yes)
-		(dnp no)
+		(dnp yes)
 		(fields_autoplaced yes)
 		(property "Reference" "R4"
